File: fpga-banks.kicad_sch (KiCad schematic)
At the start: 55 parts, among them Q17 2N7002, U21 ECP5UM5G_85_CABGA756, Y1 ECS-3225MVQ-1000CN-TR

Commit message: [#61392] Convert project to KiCad 7
[#61392] Run globlib

[#61392] Allign components to the grid

[#61392] Update oshw and antmicro logo

[#61392] Standarize ethernet sheet

[#61392] Standarize pcie-conn sheet

[#61392] Standarize rot sheet

[#61392] Standarize edge-connector sheet

[#61392] WIP:Standarize interfaces sheet

[#61392] WIP: Route interfaces sheet

[#61392] Finish standarizing interfaces sheet

[#61392] Update interfaces sheet with fixed 2N7002

[#61392] WIP:Standarize ddr3 sheet

[#61392] Standarize ddr3 sheet

[#61392] Standarize power-supply sheet

[#61392] Standarize fpga power-supply sheet

[#61392] Remove TODO comments from power-banks sheet

[#61392] Standarize fpga-banks sheet

[#61392] Ignore Input pins not driven ERC

[#61392] Clear off grid ERCs

[#61392] Exclude ERC DDR3_VTT_EN NC

[#61392] Bump rev to 1.2.1

[#61392] Bump PCB rev to 1.2.1
Parts:
- C203, C209, C219, C225, C230, C235: footprint ecp5-dc-scm-footprints:0402-cap -> antmicro-footprints:C_0402_1005Metric; symbol ecp5-dc-scm:C_4u7_0402 -> antmicroCapacitors0402:C_4u7_0402; Author (none) -> Antmicro; License (none) -> Apache-2.0; Manufacturer MURATA -> Murata; Public (none) -> False
- C204, C205, C206, C207, C210, C211, C212, C213, C214, C215, C218, C220, C221, C222, C223, C224, C226, C228, C229, C231, C232, C233, C234, C236, C237, C238, C239: footprint ecp5-dc-scm-footprints:0402-cap -> antmicro-footprints:C_0402_1005Metric; symbol ecp5-dc-scm:C_470n_0402 -> antmicroCapacitors0402:C_470n_0402; Author (none) -> Antmicro; License (none) -> Apache-2.0; Public (none) -> False
- C208, C216, C217, C241, C57, C58: footprint ecp5-dc-scm-footprints:0402-cap -> antmicro-footprints:C_0402_1005Metric; symbol ecp5-dc-scm:C_100n_0402 -> antmicroCapacitors0402:C_100n_0402; Author (none) -> Antmicro; Dielectric (none) -> X5R; License (none) -> Apache-2.0; MPN 0402X104K6R3CT -> GRM155R61H104KE14D; Manufacturer Walsin -> Murata; Public (none) -> False; Voltage (none) -> 50V
- D14, D15: footprint ecp5-dc-scm-footprints:LED_0603 -> antmicro-footprints:LED_0603_1608Metric_G; symbol ecp5-dc-scm:LG_L29K-G2J1-24-Z -> antmicroLEDIndicationDiscrete:LED_G_0603_LG_L29K-G2J1-24-Z; Author (none) -> Antmicro; Color (none) -> Green; License (none) -> Apache-2.0; Manufacturer OSRAM Opto Semiconductors Inc. -> OSRAM; Public (none) -> False
- Q17: footprint ecp5-dc-scm-footprints:SOT-23-3 -> antmicro-footprints:SOT-23-3; symbol ecp5-dc-scm:2N7002 -> antmicroTransistorsFETsMOSFETsSingle:2N7002_SOT-23-3; Author (none) -> Antmicro; License (none) -> Apache-2.0
- R126, R127, R131: footprint ecp5-dc-scm-footprints:0402-res -> antmicro-footprints:R_0402_1005Metric; symbol ecp5-dc-scm:R_10k_0402 -> antmicroResistors0402:R_10k_0402; Author (none) -> Antmicro; License (none) -> Apache-2.0; MPN CRCW040210K0FKEDHP -> CR0402-FX-1002GLF; Manufacturer VISHAY -> Bourns; Public (none) -> False; Tolerance (none) -> 1%
- R128: footprint ecp5-dc-scm-footprints:0402-res -> antmicro-footprints:R_0402_1005Metric; symbol ecp5-dc-scm:R_22R_0402 -> antmicroResistors0402:R_22R_0402; Author (none) -> Antmicro; License (none) -> Apache-2.0; MPN CRCW040222R0FKED -> CR0402-FX-22R0GLF; Manufacturer VISHAY -> Bourns; Public (none) -> False; Tolerance (none) -> 1%
- R129, R130: footprint ecp5-dc-scm-footprints:0402-res -> antmicro-footprints:R_0402_1005Metric; symbol ecp5-dc-scm:R_1k_0402 -> antmicroResistors0402:R_1k_0402; Author (none) -> Antmicro; License (none) -> Apache-2.0; Manufacturer BOURNS -> Bourns; Public (none) -> False; Tolerance (none) -> 1%
- R132, R133, R134, R135: footprint ecp5-dc-scm-footprints:0402-res -> antmicro-footprints:R_0402_1005Metric; symbol ecp5-dc-scm:R_0R_0402 -> antmicroResistors0402:R_0R_0402; Author (none) -> Antmicro; Current (none) -> 1A; DNP 1 -> (none); License (none) -> Apache-2.0; Manufacturer PANASONIC -> Panasonic; Public (none) -> False; now not fitted
- S1: footprint ecp5-dc-scm-footprints:Switch_Tactile_SMD_B3U-1000P -> antmicro-footprints:SW_B3U-1000P_SMD; symbol ecp5-dc-scm:B3U-1000P -> antmicroPushbuttonSwitches:SW_B3U-1000P_SMD; Author (none) -> Antmicro; License (none) -> Apache-2.0; Manufacturer Omron Electronics Inc-EMC Div -> Omron; Public (none) -> False
- U21: footprint ecp5-dc-scm-footprints:CABGA756_27x27mm_p0.8mm -> antmicro-footprints:BGA-1024-756_27x27mm_Layout32x32_P0.8mm; symbol ecp5-dc-scm:ECP5UM5G_85_CABGA756-ecp5-dc-scm -> antmicroFPGAChips:ECP5_LFE5UM5G-85; Author (none) -> Antmicro; License (none) -> Apache-2.0
Connections:
- net DONE: now also R128.2; no longer R128.1
- net GND: now also C231.1, C241.1; no longer C231.2, C241.2
- net INIT_N: now also D14.1 (C); no longer D14.2
- net VCC1V35: now also C231.2; no longer C231.1
- net VCC3V3: now also C241.2; no longer C241.1
- net at Q17.1 (G): now also R128.1; no longer R128.2
- net at D15.1 (C): now also Q17.3 (D); no longer R130.2
- net at D15.2 (A): now also R130.2; no longer Q17.3 (D)
- net at R129.2: now also D14.2 (A); no longer D14.1
- no-connect marks 4 -> 163
Other:
- note removed: "DNP"
- note removed: "TODO: Check and connect these misc signalls"
- moved on the sheet: C203, C204, C205, C206, C207, C208, C209, C210, C211, C212, C213, C214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

Commit message: [#61392] Import changes to the PCB
[#61392] Fix D2 orientation

[#61392] Fix J2 J1 D6 orientation

[#61392] WIP: PCB Fix caps orienations

[#61392] PCB Fix caps orienations

[#61392] Fix missalligned edge cuts

[#61392] Sync Sch with PCB

[#61392] Fix silk clipped by edge cuts

[#61392] Ignore TP no courtyard drc

[#61392] Update C_0603 footprints

[#61392] Update R_0402 footprints

[#61392] Update Sot-23 footprints

[#61392] Update QFN and IHLP footprints

[#61392] Update remaining footprints

[#61392] Change minimal text height to 0.7mm

[#61392] Clear remaining Silk DRCs

[#61392] Update TPS51200DRCT symbol

[#61392] Update 9774040151

[#61392] Update W25Q32JVS

[#61392] Update ECS-3225MVQ-1000CN-TR

[#61392] Clean ERC

[#61392] Remove obsolete files

[#61392] Synhronize components with library

[#61392] Remove globlib leftovers

[#61392] Synchronize components with libraries (WiP)

[#61392] Clean ERC and DRC

[#61392] Set J5 to DNP

[#61392] Add PCB SHA string, update layer names

[#61392] Update assets

[#62567] Add stackup.csv

[#62567] Input elecric constants for the board stackup

[#62567] Update stackup.csv
Parts:
- removed S1: B3U-1000P, antmicro-footprints:SW_B3U-1000P_SMD, symbol antmicroPushbuttonSwitches:SW_B3U-1000P_SMD
- removed Y1: ECS-3225MVQ-1000CN-TR, ecp5-dc-scm-footprints:OSC_ECS-3225MVQ-120-CN-TR, symbol ecp5-dc-scm:ECS-3225MVQ-1000CN-TR
- added SW1: SW_B3U-1000P_SMD, antmicro-footprints:SW_B3U-1000P_SMD, symbol antmicroPushbuttonSwitches:SW_B3U-1000P_SMD
- added Y1: Oscillator_100MHz_ECS_3225MV, antmicro-footprints:Oscillator_SMD_ECS_3225MV_3.2x2.5x1.2mm, symbol antmicroOscillators:Oscillator_100MHz_ECS_3225MV
- D14, D15: value LG_L29K-G2J1-24-Z -> LED_G_0603_LG_L29K-G2J1-24-Z; Public False -> (none)
- R132, R133, R134, R135: DNP (none) -> DNP; now left out of the parts list
Connections:
- net GCLK100: now also Y1.3 (OUT)
- net GND: now also SW1.2, Y1.2 (GND)
- net PROGRAM_N: now also SW1.1
- net VCC3V3: now also Y1.1 (EN), Y1.4 (VDD)
Other:
- moved on the sheet: C241
