File: interfaces.kicad_sch (KiCad schematic)
At the start: 106 parts, among them J6 10118192-0001LF, J7 61300611121, J9 0878311420, Q1 2N7002, Q2 2N7002, Q3 2N7002, U14 FT4232H-56Q, U23 ASEMB-24.000MHZ-LC-T, U24 ASEMB-24.000MHZ-LC-T, U6 MTFC16GAPALNA-AIT, U7 NVT2008DQ,115, U8 USB3300-EZK-TR, U9 USB3300-EZK-TR, Y4 ASFLMB-12.000MHZ-LC-T

Commit message: [#61392] Convert project to KiCad 7
[#61392] Run globlib

[#61392] Allign components to the grid

[#61392] Update oshw and antmicro logo

[#61392] Standarize ethernet sheet

[#61392] Standarize pcie-conn sheet

[#61392] Standarize rot sheet

[#61392] Standarize edge-connector sheet

[#61392] WIP:Standarize interfaces sheet

[#61392] WIP: Route interfaces sheet

[#61392] Finish standarizing interfaces sheet

[#61392] Update interfaces sheet with fixed 2N7002

[#61392] WIP:Standarize ddr3 sheet

[#61392] Standarize ddr3 sheet

[#61392] Standarize power-supply sheet

[#61392] Standarize fpga power-supply sheet

[#61392] Remove TODO comments from power-banks sheet

[#61392] Standarize fpga-banks sheet

[#61392] Ignore Input pins not driven ERC

[#61392] Clear off grid ERCs

[#61392] Exclude ERC DDR3_VTT_EN NC

[#61392] Bump rev to 1.2.1

[#61392] Bump PCB rev to 1.2.1
Parts:
- C227, C242, C243, C244, C245, C246, C247, C248, C249, C251, C253, C254, C255, C256, C258, C259, C51, C52, C54, C55, C60, C61, C62, C63, C64, C65, C67, C69, C71, C73, C74, C76, C98: footprint ecp5-dc-scm-footprints:0402-cap -> antmicro-footprints:C_0402_1005Metric; symbol ecp5-dc-scm:C_100n_0402 -> antmicroCapacitors0402:C_100n_0402; Author (none) -> Antmicro; Dielectric (none) -> X5R; License (none) -> Apache-2.0; MPN 0402X104K6R3CT -> GRM155R61H104KE14D; Manufacturer Walsin -> Murata; Public (none) -> False; Voltage (none) -> 50V
- C250, C252, C53, C66, C68, C70, C72, C75, C77, C99: footprint ecp5-dc-scm-footprints:0402-cap -> antmicro-footprints:C_0402_1005Metric; symbol ecp5-dc-scm:C_4u7_0402 -> antmicroCapacitors0402:C_4u7_0402; Author (none) -> Antmicro; License (none) -> Apache-2.0; Manufacturer MURATA -> Murata; Public (none) -> False
- C257: footprint ecp5-dc-scm-footprints:0603-cap -> antmicro-footprints:C_0603_1608Metric; symbol ecp5-dc-scm:C_3u3_0603 -> antmicroCapacitors0603:C_3u3_0603; Author (none) -> Antmicro; License (none) -> Apache-2.0; Public (none) -> False
- C26, C56: footprint ecp5-dc-scm-footprints:0402-cap -> antmicro-footprints:C_0402_1005Metric; symbol ecp5-dc-scm:C_10n_0402 -> antmicroCapacitors0402:C_10n_0402; Author (none) -> Antmicro; Dielectric (none) -> X7R; License (none) -> Apache-2.0; MPN 04025G103ZAT2A -> GRM155R71H103KA88D; Manufacturer AVX -> Murata; Public (none) -> False; Voltage (none) -> 50V
- C48, C49, C50: footprint ecp5-dc-scm-footprints:0603-cap -> antmicro-footprints:C_0603_1608Metric; symbol ecp5-dc-scm:C_22u_0603 -> antmicroCapacitors0603:C_22u_0603; Author (none) -> Antmicro; License (none) -> Apache-2.0; Manufacturer MURATA -> Murata; Public (none) -> False
- D2: footprint ecp5-dc-scm-footprints:SON50P350X135X55-14N -> antmicro-footprints:USON-14_3.5x1.35_P0.5mm; symbol ecp5-dc-scm:SP3011-06UTG -> antmicroTVSDiodes:SP3011-06UTG; Author (none) -> Antmicro; License (none) -> Apache-2.0; Manufacturer Littlefuse -> Littelfuse
- D3, D4, D5: value LG_L29K-G2J1-24-Z -> LED_G_0603_LG_L29K-G2J1-24-Z; footprint ecp5-dc-scm-footprints:LED_0603 -> antmicro-footprints:LED_0603_1608Metric_G; symbol ecp5-dc-scm:LG_L29K-G2J1-24-Z -> antmicroLEDIndicationDiscrete:LED_G_0603_LG_L29K-G2J1-24-Z; Author (none) -> Antmicro; Color (none) -> Green; License (none) -> Apache-2.0; Manufacturer OSRAM Opto Semiconductors Inc. -> OSRAM; Public (none) -> False
- FB10, FB9: value BLM15AG601SN1D -> FB_600Z_0.3A_Murata-BLM15AG_0402; footprint ecp5-dc-scm-footprints:0402-res -> antmicro-footprints:FB_0402_1005Metric; symbol ecp5-dc-scm:BLM15AG601SN1D -> antmicroFerriteBeadsandChips:FB_600Z_0.3A_Murata-BLM15AG_0402; Author (none) -> Antmicro; License (none) -> Apache-2.0; Public (none) -> False; Val (none) -> 600Z/0.3A
- J6: value 10118192-0001LF -> USB-Micro-B_Amphenol_10118192-0001LF; footprint ecp5-dc-scm-footprints:USB_Micro_B_Female_10118192 -> antmicro-footprints:USB-Micro-B_Receptacle_Amphenol_10118192; symbol ecp5-dc-scm:10118192-0001LF -> antmicroUSBConnectors:USB-Micro-B_Amphenol_10118192-0001LF; Author (none) -> Antmicro; License (none) -> Apache-2.0; Manufacturer Amphenol ICC (FCI) -> Amphenol
- J7: value 61300611121 -> PinHeader_1x6_P2.54mm_Drill1.1mm; footprint ecp5-dc-scm-footprints:61300611121 -> antmicro-footprints:PinHeader_1x6_P2.54mm_Drill1.1mm; symbol ecp5-dc-scm:61300611121 -> antmicroGenericPinHeaders:PinHeader_1x6_P2.54mm_Drill1.1mm; Author (none) -> Antmicro; License (none) -> Apache-2.0; Manufacturer Wurth Electronics Inc. -> Würth Elektronik
- J9: value 0878311420 -> PinHeader_2x7_P2mm_Drill1mm_Shrouded; footprint ecp5-dc-scm-footprints:PinHeader_2x7_P2mm_Drill1mm -> antmicro-footprints:PinHeader_2x7_P2mm_Drill1mm_Shrouded; symbol ecp5-dc-scm:0878311420 -> antmicroGenericPinHeaders:PinHeader_2x7_P2mm_Drill1mm_Shrouded; Author (none) -> Antmicro; License (none) -> Apache-2.0
- Q1, Q2, Q3: value 2N7002 -> 2N7002_SOT-23-3; footprint ecp5-dc-scm-footprints:SOT-23-3 -> antmicro-footprints:SOT-23-3; symbol ecp5-dc-scm:2N7002 -> antmicroTransistorsFETsMOSFETsSingle:2N7002_SOT-23-3; Author (none) -> Antmicro; License (none) -> Apache-2.0
- R14: footprint ecp5-dc-scm-footprints:0402-res -> antmicro-footprints:R_0402_1005Metric; symbol ecp5-dc-scm:R_22R_0402 -> antmicroResistors0402:R_22R_0402; Author (none) -> Antmicro; License (none) -> Apache-2.0; MPN CRCW040222R0FKED -> CR0402-FX-22R0GLF; Manufacturer VISHAY -> Bourns; Public (none) -> False; Tolerance (none) -> 1%
- R146: footprint ecp5-dc-scm-footprints:0402-res -> antmicro-footprints:R_0402_1005Metric; symbol ecp5-dc-scm:R_4k7_0402 -> antmicroResistors0402:R_4k7_0402; Author (none) -> Antmicro; License (none) -> Apache-2.0; MPN ERJ2GEJ472X -> CR0402-FX-4701GLF; Manufacturer PANASONIC_ELECTRONIC_COMPONENTS -> Bourns; Public (none) -> False; Tolerance (none) -> 1%; now not fitted
- R147: footprint ecp5-dc-scm-footprints:0402-res -> antmicro-footprints:R_0402_1005Metric; symbol ecp5-dc-scm:R_10k_0402 -> antmicroResistors0402:R_10k_0402; Author (none) -> Antmicro; License (none) -> Apache-2.0; MPN CRCW040210K0FKEDHP -> CR0402-FX-1002GLF; Manufacturer VISHAY -> Bourns; Public (none) -> False; Tolerance (none) -> 1%; now not fitted
- R148, R74, R76: footprint ecp5-dc-scm-footprints:0402-res -> antmicro-footprints:R_0402_1005Metric; symbol ecp5-dc-scm:R_1k_0402 -> antmicroResistors0402:R_1k_0402; Author (none) -> Antmicro; License (none) -> Apache-2.0; Manufacturer BOURNS -> Bourns; Public (none) -> False; Tolerance (none) -> 1%
- R149, R75, R77: footprint ecp5-dc-scm-footprints:0402-res -> antmicro-footprints:R_0402_1005Metric; symbol ecp5-dc-scm:R_12k_0402 -> antmicroResistors0402:R_12k_0402; Author (none) -> Antmicro; License (none) -> Apache-2.0; MPN CRCW040212K0FKEDHP -> CR0402-FX-1202GLF; Manufacturer VISHAY -> Bourns; Public (none) -> False; Tolerance (none) -> 1%
- R150: footprint ecp5-dc-scm-footprints:0402-res -> antmicro-footprints:R_0402_1005Metric; symbol ecp5-dc-scm:R_4k7_0402 -> antmicroResistors0402:R_4k7_0402; Author (none) -> Antmicro; License (none) -> Apache-2.0; MPN ERJ2GEJ472X -> CR0402-FX-4701GLF; Manufacturer PANASONIC_ELECTRONIC_COMPONENTS -> Bourns; Public (none) -> False; Tolerance (none) -> 1%
- R151: footprint ecp5-dc-scm-footprints:0402-res -> antmicro-footprints:R_0402_1005Metric; symbol ecp5-dc-scm:R_10k_0402 -> antmicroResistors0402:R_10k_0402; Author (none) -> Antmicro; License (none) -> Apache-2.0; MPN CRCW040210K0FKEDHP -> CR0402-FX-1002GLF; Manufacturer VISHAY -> Bourns; Public (none) -> False; Tolerance (none) -> 1%
- R49, R50, R51, R52, R53, R54, R55, R56: footprint ecp5-dc-scm-footprints:0402-res -> antmicro-footprints:R_0402_1005Metric; symbol ecp5-dc-scm:R_357k_0402 -> antmicroResistors0402:R_357k_0402; Author (none) -> Antmicro; License (none) -> Apache-2.0; MPN CRCW0402357KFKED -> CR0402-FX-3573GLF; Manufacturer Vishay -> Bourns; Public (none) -> False; Tolerance (none) -> 1%
- R57: footprint ecp5-dc-scm-footprints:0402-res -> antmicro-footprints:R_0402_1005Metric; symbol ecp5-dc-scm:R_200k_0402 -> antmicroResistors0402:R_200k_0402; Author (none) -> Antmicro; License (none) -> Apache-2.0; MPN RC0402FR-07200KL -> CR0402-FX-2003GLF; Manufacturer YAGEO_(PHYCOMP) -> Bourns; Public (none) -> False; Tolerance (none) -> 1%
- R59, R60, R61, R62, R63, R64, R65, R66, R67, R68: footprint ecp5-dc-scm-footprints:0402-res -> antmicro-footprints:R_0402_1005Metric; symbol ecp5-dc-scm:R_47k_0402 -> antmicroResistors0402:R_47k_0402; Author (none) -> Antmicro; License (none) -> Apache-2.0; MPN MCMR04X4702FTL -> CR0402-FX-4702GLF; Manufacturer MULTICOMP -> Bourns; Public (none) -> False; Tolerance (none) -> 1%
- R69, R70, R71: footprint ecp5-dc-scm-footprints:0402-res -> antmicro-footprints:R_0402_1005Metric; symbol ecp5-dc-scm:R_1k1_0402 -> antmicroResistors0402:R_1k1_0402; Author (none) -> Antmicro; License (none) -> Apache-2.0; MPN ERJ2RKF1101X -> CR0402-FX-1101GLF; Manufacturer PANASONIC_ELECTRONIC_COMPONENTS -> Bourns; Public (none) -> False; Tolerance (none) -> 1%
- U14: value FT4232H-56Q -> FT4232H_VQFN; footprint ecp5-dc-scm-footprints:QFN-56-1EP_8x8mm_P0.5mm_EP5.5.9x5.9mm -> antmicro-footprints:QFN-56-1EP_8x8mm_P0.5mm; symbol ecp5-dc-scm:FT4232H-56Q -> antmicroInterfaceControllers:FT4232H_VQFN; Author (none) -> Antmicro; License (none) -> Apache-2.0; Manufacturer FTDI -> FTDI Chip
- U6: footprint ecp5-dc-scm-footprints:BGA100CP100_17X10_1800X1400X140B46N -> antmicro-footprints:BGA-170-100_18x14mm_Layout17x10_P1mm; symbol ecp5-dc-scm:MTFC16GAPALNA-AIT -> antmicroMemory:MTFC16GAPALNA-AIT; Author (none) -> Antmicro; License (none) -> Apache-2.0; MPN (none) -> MTFC16GAPALNA-AIT; Manufacturer (none) -> Micron Technology
- U7: value NVT2008DQ,115 -> NVT2008BQ,115; footprint ecp5-dc-scm-footprints:QFN50P250X450X100-21N -> antmicro-footprints:VQFN-20_1EP_4.5x2.5mm_P0.5mm; symbol ecp5-dc-scm:NVT2008DQ,115 -> antmicroLogicTranslatorsLevelShifters:NVT2008BQ,115; Author (none) -> Antmicro; License (none) -> Apache-2.0; Manufacturer NXP Semiconductors -> NXP
- U8, U9: footprint ecp5-dc-scm-footprints:QFN50P500X500X100-33N -> antmicro-footprints:QFN-32-1EP_5x5mm; symbol ecp5-dc-scm:USB3300-EZK-TR -> antmicroInterfaceControllers:USB3300-EZK-TR; Author (none) -> Antmicro; License (none) -> Apache-2.0; Manufacturer Microchip -> Microchip Technology
- Y4: value ASFLMB-12.000MHZ-LC-T -> Oscillator_12MHz_ASFLMB; footprint ecp5-dc-scm-footprints:ASFLMB -> antmicro-footprints:Oscillator_SMD_Abracon_ASFLMB_5x3.2x0.85mm; symbol ecp5-dc-scm:ASFLMB-12.000MHZ-LC-T -> antmicroOscillators:Oscillator_12MHz_ASFLMB; Author (none) -> Antmicro; License (none) -> Apache-2.0; Manufacturer TXC -> Abracon; Public (none) -> False; Val (none) -> 12 MHz
Connections:
- net DBG_USB_D_N: now also J6.3 (D+); no longer J6.2
- net DBG_USB_D_P: now also J6.2 (D-); no longer J6.3
- net GND: now also C227.1, C242.1, C243.1, C244.1, C245.1, C246.1, C247.1, C248.1, C249.1, C250.1, C251.1, C252.1, C253.1, C254.1, C255.1, C256.1, C257.1, C258.1, C259.1, C26.1, C48.1, C49.1, C50.1, C51.1, C52.1, C53.1, C54.1, C56.1, C60.2, C61.2, C62.2, C63.2, C64.2, C65.2, C66.1, C67.2, C68.1, C69.2, C71.2, C72.1, C73.1, C75.1, C77.1, C98.1, C99.1, D2.5, U7.21 (EP); no longer C227.2, C242.2, C243.2, C244.2, C245.2, C246.2, C247.2, C248.2, C249.2, C250.2, C251.2, C252.2, C253.2, C254.2, C255.2, C256.2, C257.2, C258.2, C259.2, C26.2, C48.2, C49.2, C50.2, C51.2, C52.2, C53.2, C54.2, C56.2, C60.1, C61.1, C62.1, C63.1, C64.1, C65.1, C66.2, C67.1, C68.2, C69.1, C71.1, C72.2, C73.2, C75.2, C77.2, C98.2, C99.2
- net JTAG_TCK: now also D2.6, D2.9; no longer D2.13 (D1-)
- net JTAG_TDI: now also D2.1, D2.14; no longer D2.8 (D3-)
- net JTAG_TDO: now also D2.13, D2.2; no longer D2.9 (D3+)
- net JTAG_TMS: now also D2.7, D2.8; no longer D2.14 (D1+)
- net VBUS: now also C98.2, C99.2; no longer C98.1, C99.1
- net VCC1V0: now also C248.2; no longer C248.1
- net VCC3V3: now also C242.2, C243.2, C244.2, C245.2, C246.2, C247.2, C251.2, C253.2, C254.2, C256.2, C258.2, C26.2, C48.2, C49.2, C50.2, C51.2, C52.2, C56.2, C60.1, C61.1, C62.1, C63.1, C64.1, C65.1, C67.1, C68.2, C69.1, C72.2; no longer C242.1, C243.1, C244.1, C245.1, C246.1, C247.1, C251.1, C253.1, C254.1, C256.1, C258.1, C26.1, C48.1, C49.1, C50.1, C51.1, C52.1, C56.1, C60.2, C61.2, C62.2, C63.2, C64.2, C65.2, C67.2, C68.1, C69.2, C72.1
- net VREGOUT: now also C255.2, C257.2, C259.2; no longer C255.1, C257.1, C259.1
- net at D2.11: now also D2.4
- net at D2.12: now also D2.3
- net at FB10.2, U14.5 (V_{PHY}): now also C249.2, C252.2; no longer C249.1, C252.1
- net at FB9.2, U14.9 (V_{PLL}): now also C227.2, C250.2; no longer C227.1, C250.1
- net FTDI_CLK: now reaches U14.3 (OSCI), Y4.3 (OUT)
- net at Q1.3 (D): now also D3.1 (C); no longer D3.2
- net at R69.1: now also D3.2 (A); no longer D3.1
- net at Q2.3 (D): now also D4.1 (C); no longer D4.2
- net at R70.1: now also D4.2 (A); no longer D4.1
- net at Q3.3 (D): now also D5.1 (C); no longer D5.2
- net at R71.1: now also D5.2 (A); no longer D5.1
- net at C76.2, U9.15 (VDD1.8), U9.26 (VDD1.8): now also C77.2; no longer C77.1
- net at U8.15 (VDD1.8), U8.26 (VDD1.8): now also C71.1, C75.2; no longer C71.2, C75.1
- net 1V0_EN: no longer names the net of C55.2, R57.2, U7.19 (VREFB), U7.20 (EN)
- new net: C53.2, C54.2, U6.E4 (VDDIM)
- new net: C66.2, C73.2, U8.29 (VDDA1.8)
- no-connect marks 19 -> 43
Other:
- moved on the sheet: C227, C242, C243, C244, C245, C246, C247, C248, C249, C250, C251, C252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

Commit message: [#61392] Import changes to the PCB
[#61392] Fix D2 orientation

[#61392] Fix J2 J1 D6 orientation

[#61392] WIP: PCB Fix caps orienations

[#61392] PCB Fix caps orienations

[#61392] Fix missalligned edge cuts

[#61392] Sync Sch with PCB

[#61392] Fix silk clipped by edge cuts

[#61392] Ignore TP no courtyard drc

[#61392] Update C_0603 footprints

[#61392] Update R_0402 footprints

[#61392] Update Sot-23 footprints

[#61392] Update QFN and IHLP footprints

[#61392] Update remaining footprints

[#61392] Change minimal text height to 0.7mm

[#61392] Clear remaining Silk DRCs

[#61392] Update TPS51200DRCT symbol

[#61392] Update 9774040151

[#61392] Update W25Q32JVS

[#61392] Update ECS-3225MVQ-1000CN-TR

[#61392] Clean ERC

[#61392] Remove obsolete files

[#61392] Synhronize components with library

[#61392] Remove globlib leftovers

[#61392] Synchronize components with libraries (WiP)

[#61392] Clean ERC and DRC

[#61392] Set J5 to DNP

[#61392] Add PCB SHA string, update layer names

[#61392] Update assets

[#62567] Add stackup.csv

[#62567] Input elecric constants for the board stackup

[#62567] Update stackup.csv
Parts:
- removed TP13, TP14, TP15, TP16: TP_SMD1MM, ecp5-dc-scm-footprints:Testpoint_smd_1mm, symbol ecp5-dc-scm:TP_SMD1MM
- removed U23, U24: ASEMB-24.000MHZ-LC-T, ecp5-dc-scm-footprints:OSC_ASEM1-16.000MHZ-LC-T, symbol ecp5-dc-scm:ASEMB-24.000MHZ-LC-T
- added TP13, TP14, TP15, TP16: TP_1mm_SMD, antmicro-footprints:TP_SMD_1mm, symbol antmicroTestPoints:TP_1mm_SMD
- added Y2, Y3: Oscillator_24MHz_ASEMB, antmicro-footprints:Oscillator_SMD_Abracon_ASEMB_3.2x2.5mm, symbol antmicroOscillators:Oscillator_24MHz_ASEMB
- D3, D4, D5, Y4: Public False -> (none)
- R146, R147: now left out of the parts list
Connections:
- net DBG_USB_D_N: now also J6.2 (D-); no longer J6.3 (D+)
- net DBG_USB_D_P: now also J6.3 (D+); no longer J6.2 (D-)
- net GND: now also Y2.2 (GND), Y3.2 (GND); no longer U7.21 (EP)
- net USB1_CLK: now also Y2.3 (OUT)
- net USB2_CLK: now also Y3.3 (OUT)
- net VCC3V3: now also Y2.1 (EN), Y2.4 (VDD), Y3.1 (EN), Y3.4 (VDD)
- net at U6.K5 (DS): now also TP16.1
- net at J6.4 (ID): now also TP13.1
- net at U14.54 (~{PWR_{EN}}): now also TP14.1
- net at U14.30 (~{SUSPEND}): now also TP15.1
- no-connect marks 43 -> 44
Other:
- moved on the sheet: C26
