File: power-supply.kicad_sch (KiCad schematic)
At the start: 129 parts, among them IC1 TPS54561, J18 5040500291, J8 5040500291, Q10 2N7002, Q11 2N7002, Q12 2N7002, Q13 2N7002, Q14 2N7002, Q15 2N7002, Q16 2N7002, U12 LM3881MME_NOPB, U13 LM21212-2, U16 TPS62823DLCT, U17 TPS62823DLCT, U18 TPS62823DLCT, U19 TPS62823DLCT, U20 TPS62823DLCT

Commit message: [#61392] Convert project to KiCad 7
[#61392] Run globlib

[#61392] Allign components to the grid

[#61392] Update oshw and antmicro logo

[#61392] Standarize ethernet sheet

[#61392] Standarize pcie-conn sheet

[#61392] Standarize rot sheet

[#61392] Standarize edge-connector sheet

[#61392] WIP:Standarize interfaces sheet

[#61392] WIP: Route interfaces sheet

[#61392] Finish standarizing interfaces sheet

[#61392] Update interfaces sheet with fixed 2N7002

[#61392] WIP:Standarize ddr3 sheet

[#61392] Standarize ddr3 sheet

[#61392] Standarize power-supply sheet

[#61392] Standarize fpga power-supply sheet

[#61392] Remove TODO comments from power-banks sheet

[#61392] Standarize fpga-banks sheet

[#61392] Ignore Input pins not driven ERC

[#61392] Clear off grid ERCs

[#61392] Exclude ERC DDR3_VTT_EN NC

[#61392] Bump rev to 1.2.1

[#61392] Bump PCB rev to 1.2.1
Parts:
- removed U13: LM21212-2, ecp5-dc-scm-footprints:HTSSOP-20_TI-PWP, symbol ecp5-dc-scm:LM21212-2
- added U13: LM21212-2, antmicro-footprints:HTSSOP-20_W4.4mm_P0.65mm, symbol antmicroPMICVoltageRegulatorsDCDCSwitchingRegulators:LM21212-2
- C100, C105: footprint ecp5-dc-scm-footprints:0402-cap -> antmicro-footprints:C_0402_1005Metric; symbol ecp5-dc-scm:C_100n_0402 -> antmicroCapacitors0402:C_100n_0402; Author (none) -> Antmicro; Dielectric (none) -> X5R; License (none) -> Apache-2.0; MPN 0402X104K6R3CT -> GRM155R61H104KE14D; Manufacturer Walsin -> Murata; Public (none) -> False; Voltage (none) -> 50V
- C101, C260, C261: footprint ecp5-dc-scm-footprints:0603-cap -> antmicro-footprints:C_0603_1608Metric; symbol ecp5-dc-scm:C_10u_25V_0603 -> antmicroCapacitors0603:C_10u_25V_0603; Author (none) -> Antmicro; License (none) -> Apache-2.0; Public (none) -> False; Val 10u/25V -> 10u; Voltage (none) -> 25V
- C102: footprint ecp5-dc-scm-footprints:0402-cap -> antmicro-footprints:C_0402_1005Metric; symbol ecp5-dc-scm:C_4n7_0402 -> antmicroCapacitors0402:C_4n7_0402; Author (none) -> Antmicro; License (none) -> Apache-2.0; Public (none) -> False
- C103, C95: footprint ecp5-dc-scm-footprints:0402-cap -> antmicro-footprints:C_0402_1005Metric; symbol ecp5-dc-scm:C_10n_0402 -> antmicroCapacitors0402:C_10n_0402; Author (none) -> Antmicro; Dielectric (none) -> X7R; License (none) -> Apache-2.0; MPN 04025G103ZAT2A -> GRM155R71H103KA88D; Manufacturer AVX -> Murata; Public (none) -> False; Voltage (none) -> 50V
- C104: footprint ecp5-dc-scm-footprints:0402-cap -> antmicro-footprints:C_0402_1005Metric; symbol ecp5-dc-scm:C_47p_0402 -> antmicroCapacitors0402:C_47p_0402; Author (none) -> Antmicro; Dielectric (none) -> C0G; License (none) -> Apache-2.0; Public (none) -> False
- C106: footprint ecp5-dc-scm-footprints:0402-cap -> antmicro-footprints:C_0402_1005Metric; symbol ecp5-dc-scm:C_1n8_0402 -> antmicroCapacitors0402:C_1n8_0402; Author (none) -> Antmicro; License (none) -> Apache-2.0; Manufacturer WALSIN -> Walsin; Public (none) -> False
- C107: footprint ecp5-dc-scm-footprints:0402-cap -> antmicro-footprints:C_0402_1005Metric; symbol ecp5-dc-scm:C_180p_0402 -> antmicroCapacitors0402:C_180p_0402; Author (none) -> Antmicro; License (none) -> Apache-2.0; Public (none) -> False
- C108: footprint ecp5-dc-scm-footprints:0402-res -> antmicro-footprints:C_0402_1005Metric; symbol ecp5-dc-scm:C_750p_0402 -> antmicroCapacitors0402:C_750p_0402; Author (none) -> Antmicro; License (none) -> Apache-2.0; Public (none) -> False
- C109: footprint ecp5-dc-scm-footprints:1210-cap -> antmicro-footprints:C_1210_3225Metric; symbol ecp5-dc-scm:C_47u_1210 -> antmicroCapacitorsmisc:C_47u_1210; Author (none) -> Antmicro; License (none) -> Apache-2.0; Public (none) -> False
- C110, C111, C112: footprint ecp5-dc-scm-footprints:0603-cap -> antmicro-footprints:C_0603_1608Metric; symbol ecp5-dc-scm:C_47u_0603 -> antmicroCapacitors0603:C_47u_0603; Author (none) -> Antmicro; License (none) -> Apache-2.0; Manufacturer MURATA -> Murata; Public (none) -> False
- C113, C114, C115, C116, C117, C123, C124, C125, C126, C127, C128, C129, C130, C131, C132, C262: footprint ecp5-dc-scm-footprints:0402-cap -> antmicro-footprints:C_0402_1005Metric; symbol ecp5-dc-scm:C_10u_0402 -> antmicroCapacitors0402:C_10u_0402; Author (none) -> Antmicro; License (none) -> Apache-2.0; MPN GRM155R60J106ME44D -> CC0402MRX5R5BB106; Manufacturer MURATA -> YAGEO; Public (none) -> False
- C118, C119, C120, C121, C122: footprint ecp5-dc-scm-footprints:0402-res -> antmicro-footprints:C_0402_1005Metric; symbol ecp5-dc-scm:C_120p_0402 -> antmicroCapacitors0402:C_120p_100V_0402; Author (none) -> Antmicro; Dielectric (none) -> C0G; License (none) -> Apache-2.0; Public (none) -> False; Voltage (none) -> 100V
- C96, C97: footprint ecp5-dc-scm-footprints:0805-cap -> antmicro-footprints:C_0805_2012Metric; symbol ecp5-dc-scm:C_10u_0805 -> antmicroCapacitorsmisc:C_10u_0805; Author (none) -> Antmicro; License (none) -> Apache-2.0; Manufacturer JOHANSON_DIELECTRICS -> Johanson Technology; Public (none) -> False
- D10, D11, D12, D13, D7, D8, D9: footprint ecp5-dc-scm-footprints:LED_0603 -> antmicro-footprints:LED_0603_1608Metric_G; symbol ecp5-dc-scm:LG_L29K-G2J1-24-Z -> antmicroLEDIndicationDiscrete:LED_G_0603_LG_L29K-G2J1-24-Z; Author (none) -> Antmicro; Color (none) -> Green; License (none) -> Apache-2.0; Manufacturer OSRAM Opto Semiconductors Inc. -> OSRAM; Public (none) -> False
- D6: footprint ecp5-dc-scm-footprints:PDS760-13 -> antmicro-footprints:PowerDI5; symbol ecp5-dc-scm:PDS760-13 -> antmicroDiodesRectifiersSingle:PDS760; Author (none) -> Antmicro; License (none) -> Apache-2.0; Manufacturer Diodes Inc. -> Diodes Incorporated; Public (none) -> False
- F1: footprint ecp5-dc-scm-footprints:1206-Fuse-Littelfuse-0466-0-0-MFG -> antmicro-footprints:F_1206_3216Metric; symbol ecp5-dc-scm:0466003.NR -> antmicroFuses:F_3A_1206; Author (none) -> Antmicro; License (none) -> Apache-2.0
- L1: footprint ecp5-dc-scm-footprints:Coilcraft-XAL5030 -> antmicro-footprints:L_Coilcraft-XAL5030; symbol ecp5-dc-scm:XAL5030-801 -> antmicroFixedInductors:L_800n_13A_Coilcraft-XAL5030; Author (none) -> Antmicro; IMax (none) -> 13 A; ISat (none) -> 18.5 A; License (none) -> Apache-2.0; Public (none) -> False; Size (none) -> 5.28x5.48; Val (none) -> 800n/13A
- L2: footprint ecp5-dc-scm-footprints:WE_7447798720 -> antmicro-footprints:L_WE-PDF-1064; symbol ecp5-dc-scm:WE_7447798720 -> antmicroFixedInductors:L_7u2_7.9A_WE-PDF-1064; Author (none) -> Antmicro; IMax (none) -> 7.9 A; ISat (none) -> 6 A; License (none) -> Apache-2.0; Manufacturer Wurth Elektronik -> Würth Elektronik; Public (none) -> False; Size (none) -> 10.2x10.2; Val (none) -> 7u2/7.9A
- L3, L4, L5, L6, L7: footprint ecp5-dc-scm-footprints:IHLP-1212AE -> antmicro-footprints:L_Vishay-IHLP-1212AE; symbol ecp5-dc-scm:IHLP1212AEERR47M11 -> antmicroFixedInductors:L_470n_6.7A_Vishay-IHLP-1212AE-11; Author (none) -> Antmicro; IMax (none) -> 6.7 A; ISat (none) -> 6.7 A; License (none) -> Apache-2.0; Public (none) -> False; Size (none) -> 3.0x3.0; Val (none) -> 470n/6.7A
- Q10, Q11, Q12, Q13, Q14, Q15, Q16: footprint ecp5-dc-scm-footprints:SOT-23-3 -> antmicro-footprints:SOT-23-3; symbol ecp5-dc-scm:2N7002 -> antmicroTransistorsFETsMOSFETsSingle:2N7002_SOT-23-3; Author (none) -> Antmicro; License (none) -> Apache-2.0
- R100, R101, R102, R103, R104, R105, R106, R98: footprint ecp5-dc-scm-footprints:0402-res -> antmicro-footprints:R_0402_1005Metric; symbol ecp5-dc-scm:R_10k_0402 -> antmicroResistors0402:R_10k_0402; Author (none) -> Antmicro; License (none) -> Apache-2.0; MPN CRCW040210K0FKEDHP -> CR0402-FX-1002GLF; Manufacturer VISHAY -> Bourns; Public (none) -> False; Tolerance (none) -> 1%
- R107, R108, R109, R110, R111, R112, R113: footprint ecp5-dc-scm-footprints:0402-res -> antmicro-footprints:R_0402_1005Metric; symbol ecp5-dc-scm:R_1k_0402 -> antmicroResistors0402:R_1k_0402; Author (none) -> Antmicro; License (none) -> Apache-2.0; Manufacturer BOURNS -> Bourns; Public (none) -> False; Tolerance (none) -> 1%
- R114: footprint ecp5-dc-scm-footprints:0402-res -> antmicro-footprints:R_0402_1005Metric; symbol ecp5-dc-scm:R_453k_0402 -> antmicroResistors0402:R_453k_0402; Author (none) -> Antmicro; License (none) -> Apache-2.0; MPN CRCW0402453KFKED -> CR0402-FX-4533GLF; Manufacturer VISHAY -> Bourns; Public (none) -> False; Tolerance (none) -> 1%
- R115, R117, R119, R121, R123, R8, R85, R86, R87: footprint ecp5-dc-scm-footprints:0402-res -> antmicro-footprints:R_0402_1005Metric; symbol ecp5-dc-scm:R_100k_0402 -> antmicroResistors0402:R_100k_0402; Author (none) -> Antmicro; License (none) -> Apache-2.0; MPN CRCW0402100KFKEDHP -> CR0402-FX-1003GLF; Manufacturer VISHAY -> Bourns; Public (none) -> False; Tolerance (none) -> 1%
- R116: footprint ecp5-dc-scm-footprints:0402-res -> antmicro-footprints:R_0402_1005Metric; symbol ecp5-dc-scm:R_200k_0402 -> antmicroResistors0402:R_200k_0402; Author (none) -> Antmicro; License (none) -> Apache-2.0; MPN RC0402FR-07200KL -> CR0402-FX-2003GLF; Manufacturer YAGEO_(PHYCOMP) -> Bourns; Public (none) -> False; Tolerance (none) -> 1%
- R118: footprint ecp5-dc-scm-footprints:0402-res -> antmicro-footprints:R_0402_1005Metric; symbol ecp5-dc-scm:R_124k_0402 -> antmicroResistors0402:R_124k_0402; Author (none) -> Antmicro; License (none) -> Apache-2.0; MPN WR04X1243FTL -> CR0402-FX-1243GLF; Manufacturer WALSIN -> Bourns; Public (none) -> False; Tolerance (none) -> 1%
- R120: footprint ecp5-dc-scm-footprints:0402-res -> antmicro-footprints:R_0402_1005Metric; symbol ecp5-dc-scm:R_66k5_0402 -> antmicroResistors0402:R_66k5_0402; Author (none) -> Antmicro; License (none) -> Apache-2.0; MPN ERJ2RKF6652X -> CR0402-FX-6652GLF; Manufacturer PANASONIC -> Bourns; Public (none) -> False; Tolerance (none) -> 1%
- R137, R138, R139: footprint ecp5-dc-scm-footprints:0402-res -> antmicro-footprints:R_0402_1005Metric; symbol ecp5-dc-scm:R_0R_0402 -> antmicroResistors0402:R_0R_0402; Author (none) -> Antmicro; Current (none) -> 1A; License (none) -> Apache-2.0; Manufacturer PANASONIC -> Panasonic; Public (none) -> False
- R140, R141, R142, R143, R144, R145: footprint ecp5-dc-scm-footprints:0603-res -> antmicro-footprints:R_0603_1608Metric; symbol ecp5-dc-scm:R_0R_0603 -> antmicroResistors0603:R_0R_0603; Author (none) -> Antmicro; Current (none) -> 1A; License (none) -> Apache-2.0; Manufacturer BOURNS -> Bourns; Public (none) -> False
- R45: footprint ecp5-dc-scm-footprints:0402-res -> antmicro-footprints:R_0402_1005Metric; symbol ecp5-dc-scm:R_316k_0402 -> antmicroResistors0402:R_316k_0402; Author (none) -> Antmicro; License (none) -> Apache-2.0; MPN CRCW0402316KFKED -> CR0402-FX-3163GLF; Manufacturer VISHAY -> Bourns; Public (none) -> False; Tolerance (none) -> 1%
- R88: footprint ecp5-dc-scm-footprints:0603-res -> antmicro-footprints:R_0603_1608Metric; symbol ecp5-dc-scm:R_10R_0603 -> antmicroResistors0603:R_10R_0603; Author (none) -> Antmicro; License (none) -> Apache-2.0; MPN MCWR06X10R0FTL -> CR0603-FX-10R0ELF; Manufacturer MULTICOMP -> Bourns; Public (none) -> False; Tolerance (none) -> 1%
- R89: footprint ecp5-dc-scm-footprints:0402-res -> antmicro-footprints:R_0402_1005Metric; symbol ecp5-dc-scm:R_47k_0402 -> antmicroResistors0402:R_47k_0402; Author (none) -> Antmicro; License (none) -> Apache-2.0; MPN MCMR04X4702FTL -> CR0402-FX-4702GLF; Manufacturer MULTICOMP -> Bourns; Public (none) -> False; Tolerance (none) -> 1%
- R90: footprint ecp5-dc-scm-footprints:0402-res -> antmicro-footprints:R_0402_1005Metric; symbol ecp5-dc-scm:R_16k9_0402 -> antmicroResistors0402:R_16k9_0402; Author (none) -> Antmicro; License (none) -> Apache-2.0; MPN ERA2AEB1692X -> CR0402-FX-1692GLF; Manufacturer PANASONIC -> Bourns; Public (none) -> False; Tolerance (none) -> 1%
- R91: footprint ecp5-dc-scm-footprints:0402-res -> antmicro-footprints:R_0402_1005Metric; symbol ecp5-dc-scm:R_243k_0402 -> antmicroResistors0402:R_243k_0402; Author (none) -> Antmicro; License (none) -> Apache-2.0; MPN MCMR04X2433FTL -> CR0402-FX-2433GLF; Manufacturer MULTICOMP -> Bourns; Public (none) -> False; Tolerance (none) -> 1%
- R93: footprint ecp5-dc-scm-footprints:0402-res -> antmicro-footprints:R_0402_1005Metric; symbol ecp5-dc-scm:R_4k7_0402 -> antmicroResistors0402:R_4k7_0402; Author (none) -> Antmicro; License (none) -> Apache-2.0; MPN ERJ2GEJ472X -> CR0402-FX-4701GLF; Manufacturer PANASONIC_ELECTRONIC_COMPONENTS -> Bourns; Public (none) -> False; Tolerance (none) -> 1%
- R94: footprint ecp5-dc-scm-footprints:1206-res -> antmicro-footprints:R_1206_3216Metric; symbol ecp5-dc-scm:R_0R_1206 -> antmicroResistorsmisc:R_0R_1206; Author (none) -> Antmicro; Current (none) -> 2A; License (none) -> Apache-2.0; Manufacturer MULTICOMP -> Multicomp Pro; Public (none) -> False
- R95: footprint ecp5-dc-scm-footprints:0402-res -> antmicro-footprints:R_0402_1005Metric; symbol ecp5-dc-scm:R_49R9_0402 -> antmicroResistors0402:R_49R9_0402; Author (none) -> Antmicro; License (none) -> Apache-2.0; MPN CRCW040249R9FKED -> CR0402-FX-49R9GLF; Manufacturer VISHAY -> Bourns; Public (none) -> False; Tolerance (none) -> 1%
- R96: footprint ecp5-dc-scm-footprints:0402-res -> antmicro-footprints:R_0402_1005Metric; symbol ecp5-dc-scm:R_53k6_0402 -> antmicroResistors0402:R_53k6_0402; Author (none) -> Antmicro; License (none) -> Apache-2.0; MPN CPF0402B53K6E1_ -> CR0402-FX-5362GLF; Manufacturer TE_CONNECTIVITY -> Bourns; Public (none) -> False; Tolerance (none) -> 1%
- R97: footprint ecp5-dc-scm-footprints:0402-res -> antmicro-footprints:R_0402_1005Metric; symbol ecp5-dc-scm:R_10k2_0402 -> antmicroResistors0402:R_10k2_0402; Author (none) -> Antmicro; License (none) -> Apache-2.0; MPN MCWR04X1022FTL -> CR0402-FX-1022GLF; Manufacturer MULTICOMP -> Bourns; Public (none) -> False; Tolerance (none) -> 1%
- R99: footprint ecp5-dc-scm-footprints:0402-res -> antmicro-footprints:R_0402_1005Metric; symbol ecp5-dc-scm:R_470k_0402 -> antmicroResistors0402:R_470k_0402; Author (none) -> Antmicro; License (none) -> Apache-2.0; MPN RC0402FR-07470KL -> CR0402-FX-4703GLF; Manufacturer YAGEO -> Bourns; Public (none) -> False; Tolerance (none) -> 1%
- TP4, TP5: footprint ecp5-dc-scm-footprints:PROBE_PAD_1206 -> antmicro-footprints:TP_1206_SMD_RCW-0C; symbol ecp5-dc-scm:RCW-0C -> antmicroTestPoints:TP_1206_SMD_RCW-0C; Author (none) -> Antmicro; License (none) -> Apache-2.0; Manufacturer TE Connectivity AMP Connectors -> TE Connectivity
- U12: footprint ecp5-dc-scm-footprints:VSSOP8-Texas_Instruments-DGK0008A -> antmicro-footprints:VSSOP-8_3x3mm_P0.65mm; symbol ecp5-dc-scm:LM3881MME_NOPB -> antmicroPMICPowerSequencers:LM3881; Author (none) -> Antmicro; License (none) -> Apache-2.0
- U16, U17, U18, U19, U20: footprint ecp5-dc-scm-footprints:QFN-8_2x1mm -> antmicro-footprints:QFN-8_2x1.5mm; symbol ecp5-dc-scm:TPS62823DLCT -> antmicroDCDCConverters:TPS62823DLCT; Author (none) -> Antmicro; License (none) -> Apache-2.0
Connections:
- net 1V2_PG: now also U13.17 (PGOOD)
- net 5V0_PG: now also C262.2; no longer C262.1
- net GND: now also C100.1, C101.1, C102.1, C103.1, C104.1, C109.1, C113.1, C115.1, C116.1, C117.1, C123.1, C124.1, C125.1, C126.1, C127.1, C128.1, C129.1, C130.1, C131.1, C132.1, C260.1, C261.1, C262.1, C95.1, C96.1, C97.1, D6.2 (A), U13.10 (PGND), U13.20 (AGND), U13.21 (EP), U13.8 (PGND), U13.9 (PGND); no longer C100.2, C101.2, C102.2, C103.2, C104.2, C109.2, C110.2, C111.2, C112.2, C113.2, C115.2, C116.2, C117.2, C123.2, C124.2, C125.2, C126.2, C127.2, C128.2, C129.2, C130.2, C131.2, C132.2, C260.2, C261.2, C262.2, C95.2, C96.2, C97.2, D6.A
- net VCC12V: now also C101.2, C260.2, C261.2; no longer C101.1, C260.1, C261.1
- net VCC5V0: now also C113.2, C115.2, C116.2, C117.2, C96.2, C97.2, U13.5 (PVIN), U13.6 (PVIN), U13.7 (PVIN); no longer C113.1, C115.1, C116.1, C117.1, C96.1, C97.1
- net VCCA0_EN: now also U13.3 (EN)
- net at L2.2, R94.2, R95.1: now also C110.2, C111.2, C112.2; no longer C110.1, C111.1, C112.1
- net at R123.1, R45.1, U16.2 (FB): now also C122.1; no longer C122.2
- net at L7.2, R145.2, R45.2: now also C122.2, C127.2, C132.2; no longer C122.1, C127.1, C132.1
- net at R88.2: now also C100.2, U13.4 (AVIN); no longer C100.1
- net at R89.1: now also U13.1 (FADJ)
- net at L1.2, R140.2, R98.1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: now also C108.2, C109.2; no longer C108.1, C109.1
- net at C106.1: now also C107.1, U13.18 (COMP); no longer R93.1
- net at C106.2: now also R93.1; no longer C107.2
- net at R100.1, R93.2, R98.2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: now also C107.2, U13.19 (FB); no longer C107.1
- net at R99.1: now also C108.1; no longer C108.2
- net at L1.1: now also U13.11 (SW), U13.12 (SW), U13.13 (SW), U13.14 (SW), U13.15 (SW), U13.16 (SW)
- net at R120.1, R121.1, U20.2 (FB): now also C121.1; no longer C121.2
- net at L6.2, R120.2, R144.2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: now also C121.2, C126.2, C131.2; no longer C121.1, C126.1, C131.1
- net at IC1.1 (BOOT): now also C105.1; no longer C105.2
- net at IC1.4 (SS/TR): now also C103.2; no longer C103.1
- net at IC1.7 (COMP), R90.1: now also C104.2; no longer C104.1
- net at IC1.9 (SW), L2.1: now also C105.2, D6.1 (C); no longer C105.1, D6.C
- net at R90.2: now also C102.2; no longer C102.1
- net at U12.5 (TADJ): now also C95.2; no longer C95.1
- net at R114.2, R115.1, U17.2 (FB): now also C118.1; no longer C118.2
- net at L3.2, R114.1, R141.2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: now also C118.2, C123.2, C128.2; no longer C118.1, C123.1, C128.1
- net at R116.2, R117.1, U18.2 (FB): now also C119.1; no longer C119.2
- net at L4.2, R116.1, R142.2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: now also C119.2, C124.2, C129.2; no longer C119.1, C124.1, C129.1
- net at R118.2, R119.1, U19.2 (FB): now also C120.1; no longer C120.2
- net at L5.2, R118.1, R143.2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: now also C120.2, C125.2, C130.2; no longer C120.1, C125.1, C130.1
- new net: C110.1, C111.1, C112.1
- no-connect marks 2 -> 1
Other:
- moved on the sheet: C100, C101, C102, C103, C104, C105, C106, C107, C108, C109, C110, C111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

Commit message: [#61392] Import changes to the PCB
[#61392] Fix D2 orientation

[#61392] Fix J2 J1 D6 orientation

[#61392] WIP: PCB Fix caps orienations

[#61392] PCB Fix caps orienations

[#61392] Fix missalligned edge cuts

[#61392] Sync Sch with PCB

[#61392] Fix silk clipped by edge cuts

[#61392] Ignore TP no courtyard drc

[#61392] Update C_0603 footprints

[#61392] Update R_0402 footprints

[#61392] Update Sot-23 footprints

[#61392] Update QFN and IHLP footprints

[#61392] Update remaining footprints

[#61392] Change minimal text height to 0.7mm

[#61392] Clear remaining Silk DRCs

[#61392] Update TPS51200DRCT symbol

[#61392] Update 9774040151

[#61392] Update W25Q32JVS

[#61392] Update ECS-3225MVQ-1000CN-TR

[#61392] Clean ERC

[#61392] Remove obsolete files

[#61392] Synhronize components with library

[#61392] Remove globlib leftovers

[#61392] Synchronize components with libraries (WiP)

[#61392] Clean ERC and DRC

[#61392] Set J5 to DNP

[#61392] Add PCB SHA string, update layer names

[#61392] Update assets

[#62567] Add stackup.csv

[#62567] Input elecric constants for the board stackup

[#62567] Update stackup.csv
Parts:
- removed C103: C_10n_0402, antmicro-footprints:C_0402_1005Metric, symbol antmicroCapacitors0402:C_10n_0402
- removed IC1: TPS54561, ecp5-dc-scm-footprints:WSON-10_4x4, symbol ecp5-dc-scm:TPS54561
- removed J18, J8: 5040500291, ecp5-dc-scm-footprints:MOLEX_5040500291, symbol ecp5-dc-scm:5040500291
- removed TP10, TP11, TP12, TP6, TP7, TP8, TP9: TP_SMD1MM, ecp5-dc-scm-footprints:Testpoint_smd_1mm, symbol ecp5-dc-scm:TP_SMD1MM
- added C59: C_10n_0402, antmicro-footprints:C_0402_1005Metric, symbol antmicroCapacitors0402:C_10n_0402
- added J18, J8: Molex_Pico-Lock_1x2_504050-0291, antmicro-footprints:Conn_Molex_Pico-Lock_1x2_504050-0291, symbol antmicroWire2BoardConnectors:Molex_Pico-Lock_1x2_504050-0291
- added TP10, TP11, TP12, TP6, TP7, TP8, TP9: TP_1mm_SMD, antmicro-footprints:TP_SMD_1mm, symbol antmicroTestPoints:TP_1mm_SMD
- added U15: TPS54561QDPRRQ1, antmicro-footprints:WSON-10-1EP_4x4mm_P0.8mm_EP2.6x3mm, symbol antmicroPMICVoltageRegulatorsLinear:TPS54561QDPRRQ1
- D10, D11, D12, D13, D7, D8, D9: value LG_L29K-G2J1-24-Z -> LED_G_0603_LG_L29K-G2J1-24-Z; Public False -> (none)
- D6: value PDS760-13 -> PDS760; Public False -> (none)
Connections:
- net 3V0_BAT: now also J18.1
- net 5V0_PG: now also TP12.1, U15.10 (PWRGD)
- net GND: now also C110.1, C111.1, C112.1, R121.1, C59.1, J18.2, J18.SH, J8.2, J8.SH, U15.11 (GND), U15.8 (GND); no longer R121.2
- net P12V_AUX: now also J8.1
- net VCC12V: now also U15.2 (V_{DD})
- net at C108.2, C109.2, L1.2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: now also TP7.1
- net at C121.1, R120.1, U20.2 (FB): now also R121.2; no longer R121.1
- net at C121.2, C126.2, C131.2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: now also TP11.1
- net at C105.1: now also U15.1 (BOOT)
- net at R91.2: now also U15.5 (RT/CLK)
- net at R96.2, R97.1: now also U15.6 (FB)
- net at C104.2, R90.1: now also U15.7 (COMP)
- net at C105.2, D6.1 (C), L2.1: now also U15.9 (SW)
- net at C118.2, C123.2, C128.2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: now also TP8.1
- net at C119.2, C124.2, C129.2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: now also TP9.1
- net at C120.2, C125.2, C130.2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: now also TP10.1
- new net: TP6.1, U15.3 (EN)
- new net: C59.2, U15.4 (SS/TR)
Other:
- moved on the sheet: C102, C104, C105, C110, C111, C112, C114, C118, C123, C128, L2, L3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
